Commit message: update from kinova-ros

File: kinova-ros/kinova_description/urdf/j2n4s300.xacro (robot description, xacro)
@@ -71,5 +71,5 @@
     <xacro:property name="joint_end_effector_axis_xyz" value="0 0 0" />
     <xacro:property name="joint_end_effector_origin_xyz" value="0 0 -0.1600" />
-    <xacro:property name="joint_end_effector_origin_rpy" value="${J_PI} 0 0" />
+    <xacro:property name="joint_end_effector_origin_rpy" value="${J_PI} 0 ${J_PI/2}" />
     <xacro:macro name="j2n4s300" params="base_parent prefix:=j2n4s300">
         <xacro:gazebo_config robot_namespace="${prefix}"/>
@@ -82,5 +82,5 @@
         <xacro:kinova_armlink link_name="${prefix}_link_3" link_mesh="${link_3_mesh}" use_ring_mesh="true" mesh_no="${link_3_mesh_no}"/>
         <xacro:kinova_armjoint joint_name="${prefix}_joint_3" type="${joint_3_type}" parent="${prefix}_link_2" child="${prefix}_link_3" joint_axis_xyz="${joint_3_axis_xyz}" joint_origin_xyz="${joint_3_origin_xyz}" joint_origin_rpy="${joint_3_origin_rpy}" joint_lower_limit="${joint_3_lower_limit}" joint_upper_limit="${joint_3_upper_limit}"/>
-        <xacro:kinova_armlink link_name="${prefix}_link_4" link_mesh="${link_4_mesh}" use_ring_mesh="true" ring_mesh="ring_small"/>
+        <xacro:kinova_armlink link_name="${prefix}_link_4" link_mesh="${link_4_mesh}" use_ring_mesh="true" ring_mesh="ring_small" mesh_no="${link_4_mesh_no}"/>
         <xacro:kinova_armjoint joint_name="${prefix}_joint_4" type="${joint_4_type}" parent="${prefix}_link_3" child="${prefix}_link_4" joint_axis_xyz="${joint_4_axis_xyz}" joint_origin_xyz="${joint_4_origin_xyz}" joint_origin_rpy="${joint_4_origin_rpy}" joint_lower_limit="${joint_4_lower_limit}" joint_upper_limit="${joint_4_upper_limit}"/>
         <xacro:kinova_virtual_link link_name="${prefix}_end_effector"/>

File: kinova-ros/kinova_description/urdf/j2n4s300_standalone.xacro (robot description, xacro)
@@ -3,38 +3,17 @@
 <robot xmlns:xi="http://www.w3.org/2001/XInclude"
 	xmlns:gazebo="http://playerstage.sourceforge.net/gazebo/xmlschema/#gz"
-	xmlns:model="http://playerstage.sourceforge.net/gazebo/xmlschema/#model"
+    xmlns:model="http://playerstage.sourceforge.net/gazebo/xmlschema/#model"
 	xmlns:sensor="http://playerstage.sourceforge.net/gazebo/xmlschema/#sensor"
 	xmlns:body="http://playerstage.sourceforge.net/gazebo/xmlschema/#body"
-	xmlns:geom="http://playerstage.sourceforge.net/gazebo/xmlschema/#geom"
-	xmlns:joint="http://playerstage.sourceforge.net/gazebo/xmlschema/#joint"
+    xmlns:geom="http://playerstage.sourceforge.net/gazebo/xmlschema/#geom"
+    xmlns:joint="http://playerstage.sourceforge.net/gazebo/xmlschema/#joint"
 	xmlns:controller="http://playerstage.sourceforge.net/gazebo/xmlschema/#controller"
 	xmlns:interface="http://playerstage.sourceforge.net/gazebo/xmlschema/#interface"
 	xmlns:rendering="http://playerstage.sourceforge.net/gazebo/xmlschema/#rendering"
-	xmlns:renderable="http://playerstage.sourceforge.net/gazebo/xmlschema/#renderable"
-	xmlns:physics="http://playerstage.sourceforge.net/gazebo/xmlschema/#physics"
+    xmlns:renderable="http://playerstage.sourceforge.net/gazebo/xmlschema/#renderable"
+    xmlns:physics="http://playerstage.sourceforge.net/gazebo/xmlschema/#physics"
 	xmlns:xacro="http://ros.org/wiki/xacro" name="j2n4s300">
   <xacro:include filename="$(find kinova_description)/urdf/j2n4s300.xacro"/>
-  <link name="root">
-    <visual>
-      <origin xyz="0 0 0" rpy="0 0 0" />
-      <geometry>
-        <box size = "0.01 0.01 0.01"/>
-      </geometry>
-    <!--<material name="Black" /> -->
-    </visual>
-    <collision>
-      <origin xyz="0 0 0" rpy="0 0 0" />
-      <geometry>
-        <box size = "0.01 0.01 0.01"/>
-      </geometry>
-    </collision>
-  </link>
-  <!-- for gazebo -->
-  <link name="world"/>
-  <joint name="connect_root_and_world" type="fixed">
-    <child link="root" />
-    <parent link="world" />
-    <origin xyz="0 0 0" rpy="0 0 0" />
-  </joint>
+  <link name="root" />
   <xacro:property name="robot_root" value="root" />
   <xacro:j2n4s300  base_parent="${robot_root}"/>

File: kinova-ros/kinova_description/urdf/j2n6s200_standalone.xacro (robot description, xacro)
@@ -3,38 +3,17 @@
 <robot xmlns:xi="http://www.w3.org/2001/XInclude"
 	xmlns:gazebo="http://playerstage.sourceforge.net/gazebo/xmlschema/#gz"
-	xmlns:model="http://playerstage.sourceforge.net/gazebo/xmlschema/#model"
+    xmlns:model="http://playerstage.sourceforge.net/gazebo/xmlschema/#model"
 	xmlns:sensor="http://playerstage.sourceforge.net/gazebo/xmlschema/#sensor"
 	xmlns:body="http://playerstage.sourceforge.net/gazebo/xmlschema/#body"
-	xmlns:geom="http://playerstage.sourceforge.net/gazebo/xmlschema/#geom"
-	xmlns:joint="http://playerstage.sourceforge.net/gazebo/xmlschema/#joint"
+    xmlns:geom="http://playerstage.sourceforge.net/gazebo/xmlschema/#geom"
+    xmlns:joint="http://playerstage.sourceforge.net/gazebo/xmlschema/#joint"
 	xmlns:controller="http://playerstage.sourceforge.net/gazebo/xmlschema/#controller"
 	xmlns:interface="http://playerstage.sourceforge.net/gazebo/xmlschema/#interface"
 	xmlns:rendering="http://playerstage.sourceforge.net/gazebo/xmlschema/#rendering"
-	xmlns:renderable="http://playerstage.sourceforge.net/gazebo/xmlschema/#renderable"
-	xmlns:physics="http://playerstage.sourceforge.net/gazebo/xmlschema/#physics"
+    xmlns:renderable="http://playerstage.sourceforge.net/gazebo/xmlschema/#renderable"
+    xmlns:physics="http://playerstage.sourceforge.net/gazebo/xmlschema/#physics"
 	xmlns:xacro="http://ros.org/wiki/xacro" name="j2n6s200">
   <xacro:include filename="$(find kinova_description)/urdf/j2n6s200.xacro"/>
-  <link name="root">
-    <visual>
-      <origin xyz="0 0 0" rpy="0 0 0" />
-      <geometry>
-        <box size = "0.01 0.01 0.01"/>
-      </geometry>
-    <!--<material name="Black" /> -->
-    </visual>
-    <collision>
-      <origin xyz="0 0 0" rpy="0 0 0" />
-      <geometry>
-        <box size = "0.01 0.01 0.01"/>
-      </geometry>
-    </collision>
-  </link>
-  <!-- for gazebo -->
-  <link name="world"/>
-  <joint name="connect_root_and_world" type="fixed">
-    <child link="root" />
-    <parent link="world" />
-    <origin xyz="0 0 0" rpy="0 0 0" />
-  </joint>
+  <link name="root"/>
   <xacro:property name="robot_root" value="root" />
   <xacro:j2n6s200  base_parent="${robot_root}"/>

File: kinova-ros/kinova_description/urdf/j2n6s300_standalone.xacro (robot description, xacro)
@@ -3,38 +3,17 @@
 <robot xmlns:xi="http://www.w3.org/2001/XInclude"
 	xmlns:gazebo="http://playerstage.sourceforge.net/gazebo/xmlschema/#gz"
-	xmlns:model="http://playerstage.sourceforge.net/gazebo/xmlschema/#model"
+    xmlns:model="http://playerstage.sourceforge.net/gazebo/xmlschema/#model"
 	xmlns:sensor="http://playerstage.sourceforge.net/gazebo/xmlschema/#sensor"
 	xmlns:body="http://playerstage.sourceforge.net/gazebo/xmlschema/#body"
-	xmlns:geom="http://playerstage.sourceforge.net/gazebo/xmlschema/#geom"
-	xmlns:joint="http://playerstage.sourceforge.net/gazebo/xmlschema/#joint"
+    xmlns:geom="http://playerstage.sourceforge.net/gazebo/xmlschema/#geom"
+    xmlns:joint="http://playerstage.sourceforge.net/gazebo/xmlschema/#joint"
 	xmlns:controller="http://playerstage.sourceforge.net/gazebo/xmlschema/#controller"
 	xmlns:interface="http://playerstage.sourceforge.net/gazebo/xmlschema/#interface"
 	xmlns:rendering="http://playerstage.sourceforge.net/gazebo/xmlschema/#rendering"
-	xmlns:renderable="http://playerstage.sourceforge.net/gazebo/xmlschema/#renderable"
-	xmlns:physics="http://playerstage.sourceforge.net/gazebo/xmlschema/#physics"
+    xmlns:renderable="http://playerstage.sourceforge.net/gazebo/xmlschema/#renderable"
+    xmlns:physics="http://playerstage.sourceforge.net/gazebo/xmlschema/#physics"
 	xmlns:xacro="http://ros.org/wiki/xacro" name="j2n6s300">
   <xacro:include filename="$(find kinova_description)/urdf/j2n6s300.xacro"/>
-  <link name="root">
-    <visual>
-      <origin xyz="0 0 0" rpy="0 0 0" />
-      <geometry>
-        <box size = "0.01 0.01 0.01"/>
-      </geometry>
-    <!--<material name="Black" /> -->
-    </visual>
-    <collision>
-      <origin xyz="0 0 0" rpy="0 0 0" />
-      <geometry>
-        <box size = "0.01 0.01 0.01"/>
-      </geometry>
-    </collision>
-  </link>
-  <!-- for gazebo -->
-  <link name="world"/>
-  <joint name="connect_root_and_world" type="fixed">
-    <child link="root" />
-    <parent link="world" />
-    <origin xyz="0 0 0" rpy="0 0 0" />
-  </joint>
+  <link name="root"/>
   <xacro:property name="robot_root" value="root" />
   <xacro:j2n6s300  base_parent="${robot_root}"/>

File: kinova-ros/kinova_description/urdf/j2n7s300_standalone.xacro (robot description, xacro)
@@ -3,38 +3,17 @@
 <robot xmlns:xi="http://www.w3.org/2001/XInclude"
 	xmlns:gazebo="http://playerstage.sourceforge.net/gazebo/xmlschema/#gz"
-	xmlns:model="http://playerstage.sourceforge.net/gazebo/xmlschema/#model"
+    xmlns:model="http://playerstage.sourceforge.net/gazebo/xmlschema/#model"
 	xmlns:sensor="http://playerstage.sourceforge.net/gazebo/xmlschema/#sensor"
 	xmlns:body="http://playerstage.sourceforge.net/gazebo/xmlschema/#body"
-	xmlns:geom="http://playerstage.sourceforge.net/gazebo/xmlschema/#geom"
-	xmlns:joint="http://playerstage.sourceforge.net/gazebo/xmlschema/#joint"
+    xmlns:geom="http://playerstage.sourceforge.net/gazebo/xmlschema/#geom"
+    xmlns:joint="http://playerstage.sourceforge.net/gazebo/xmlschema/#joint"
 	xmlns:controller="http://playerstage.sourceforge.net/gazebo/xmlschema/#controller"
 	xmlns:interface="http://playerstage.sourceforge.net/gazebo/xmlschema/#interface"
 	xmlns:rendering="http://playerstage.sourceforge.net/gazebo/xmlschema/#rendering"
-	xmlns:renderable="http://playerstage.sourceforge.net/gazebo/xmlschema/#renderable"
-	xmlns:physics="http://playerstage.sourceforge.net/gazebo/xmlschema/#physics"
+    xmlns:renderable="http://playerstage.sourceforge.net/gazebo/xmlschema/#renderable"
+    xmlns:physics="http://playerstage.sourceforge.net/gazebo/xmlschema/#physics"
 	xmlns:xacro="http://ros.org/wiki/xacro" name="j2n7s300">
   <xacro:include filename="$(find kinova_description)/urdf/j2n7s300.xacro"/>
-  <link name="root">
-    <visual>
-      <origin xyz="0 0 0" rpy="0 0 0" />
-      <geometry>
-        <box size = "0.01 0.01 0.01"/>
-      </geometry>
-    <!--<material name="Black" /> -->
-    </visual>
-    <collision>
-      <origin xyz="0 0 0" rpy="0 0 0" />
-      <geometry>
-        <box size = "0.01 0.01 0.01"/>
-      </geometry>
-    </collision>
-  </link>
-  <!-- for gazebo -->
-  <link name="world"/>
-  <joint name="connect_root_and_world" type="fixed">
-    <child link="root" />
-    <parent link="world" />
-    <origin xyz="0 0 0" rpy="0 0 0" />
-  </joint>
+  <link name="root"/>
   <xacro:property name="robot_root" value="root" />
   <xacro:j2n7s300  base_parent="${robot_root}"/>

File: kinova-ros/kinova_description/urdf/j2s6s300_standalone.xacro (robot description, xacro)
@@ -3,38 +3,17 @@
 <robot xmlns:xi="http://www.w3.org/2001/XInclude"
 	xmlns:gazebo="http://playerstage.sourceforge.net/gazebo/xmlschema/#gz"
-	xmlns:model="http://playerstage.sourceforge.net/gazebo/xmlschema/#model"
+    xmlns:model="http://playerstage.sourceforge.net/gazebo/xmlschema/#model"
 	xmlns:sensor="http://playerstage.sourceforge.net/gazebo/xmlschema/#sensor"
 	xmlns:body="http://playerstage.sourceforge.net/gazebo/xmlschema/#body"
-	xmlns:geom="http://playerstage.sourceforge.net/gazebo/xmlschema/#geom"
-	xmlns:joint="http://playerstage.sourceforge.net/gazebo/xmlschema/#joint"
+    xmlns:geom="http://playerstage.sourceforge.net/gazebo/xmlschema/#geom"
+    xmlns:joint="http://playerstage.sourceforge.net/gazebo/xmlschema/#joint"
 	xmlns:controller="http://playerstage.sourceforge.net/gazebo/xmlschema/#controller"
 	xmlns:interface="http://playerstage.sourceforge.net/gazebo/xmlschema/#interface"
 	xmlns:rendering="http://playerstage.sourceforge.net/gazebo/xmlschema/#rendering"
-	xmlns:renderable="http://playerstage.sourceforge.net/gazebo/xmlschema/#renderable"
-	xmlns:physics="http://playerstage.sourceforge.net/gazebo/xmlschema/#physics"
+    xmlns:renderable="http://playerstage.sourceforge.net/gazebo/xmlschema/#renderable"
+    xmlns:physics="http://playerstage.sourceforge.net/gazebo/xmlschema/#physics"
 	xmlns:xacro="http://ros.org/wiki/xacro" name="j2s6s300">
   <xacro:include filename="$(find kinova_description)/urdf/j2s6s300.xacro"/>
-  <link name="root">
-    <visual>
-      <origin xyz="0 0 0" rpy="0 0 0" />
-      <geometry>
-        <box size = "0.01 0.01 0.01"/>
-      </geometry>
-    <!--<material name="Black" /> -->
-    </visual>
-    <collision>
-      <origin xyz="0 0 0" rpy="0 0 0" />
-      <geometry>
-        <box size = "0.01 0.01 0.01"/>
-      </geometry>
-    </collision>
-  </link>
-  <!-- for gazebo -->
-  <link name="world"/>
-  <joint name="connect_root_and_world" type="fixed">
-    <child link="root" />
-    <parent link="world" />
-    <origin xyz="0 0 0" rpy="0 0 0" />
-  </joint>
+  <link name="root"/>
   <xacro:property name="robot_root" value="root" />
   <xacro:j2s6s300  base_parent="${robot_root}"/>

File: kinova-ros/kinova_description/urdf/j2s7s300_standalone.xacro (robot description, xacro)
@@ -3,38 +3,17 @@
 <robot xmlns:xi="http://www.w3.org/2001/XInclude"
 	xmlns:gazebo="http://playerstage.sourceforge.net/gazebo/xmlschema/#gz"
-	xmlns:model="http://playerstage.sourceforge.net/gazebo/xmlschema/#model"
+    xmlns:model="http://playerstage.sourceforge.net/gazebo/xmlschema/#model"
 	xmlns:sensor="http://playerstage.sourceforge.net/gazebo/xmlschema/#sensor"
 	xmlns:body="http://playerstage.sourceforge.net/gazebo/xmlschema/#body"
-	xmlns:geom="http://playerstage.sourceforge.net/gazebo/xmlschema/#geom"
-	xmlns:joint="http://playerstage.sourceforge.net/gazebo/xmlschema/#joint"
+    xmlns:geom="http://playerstage.sourceforge.net/gazebo/xmlschema/#geom"
+    xmlns:joint="http://playerstage.sourceforge.net/gazebo/xmlschema/#joint"
 	xmlns:controller="http://playerstage.sourceforge.net/gazebo/xmlschema/#controller"
 	xmlns:interface="http://playerstage.sourceforge.net/gazebo/xmlschema/#interface"
 	xmlns:rendering="http://playerstage.sourceforge.net/gazebo/xmlschema/#rendering"
-	xmlns:renderable="http://playerstage.sourceforge.net/gazebo/xmlschema/#renderable"
-	xmlns:physics="http://playerstage.sourceforge.net/gazebo/xmlschema/#physics"
+    xmlns:renderable="http://playerstage.sourceforge.net/gazebo/xmlschema/#renderable"
+    xmlns:physics="http://playerstage.sourceforge.net/gazebo/xmlschema/#physics"
 	xmlns:xacro="http://ros.org/wiki/xacro" name="j2s7s300">
   <xacro:include filename="$(find kinova_description)/urdf/j2s7s300.xacro"/>
-  <link name="root">
-    <visual>
-      <origin xyz="0 0 0" rpy="0 0 0" />
-      <geometry>
-        <box size = "0.01 0.01 0.01"/>
-      </geometry>
-    <!--<material name="Black" /> -->
-    </visual>
-    <collision>
-      <origin xyz="0 0 0" rpy="0 0 0" />
-      <geometry>
-        <box size = "0.01 0.01 0.01"/>
-      </geometry>
-    </collision>
-  </link>
-  <!-- for gazebo -->
-  <link name="world"/>
-  <joint name="connect_root_and_world" type="fixed">
-    <child link="root" />
-    <parent link="world" />
-    <origin xyz="0 0 0" rpy="0 0 0" />
-  </joint>
+  <link name="root"/>
   <xacro:property name="robot_root" value="root" />
   <xacro:j2s7s300  base_parent="${robot_root}"/>

File: kinova-ros/kinova_description/urdf/kinova_common.xacro (robot description, xacro)
@@ -2,14 +2,14 @@
 <root xmlns:xi="http://www.w3.org/2001/XInclude"
 	xmlns:gazebo="http://playerstage.sourceforge.net/gazebo/xmlschema/#gz"
-	xmlns:model="http://playerstage.sourceforge.net/gazebo/xmlschema/#model"
+    xmlns:model="http://playerstage.sourceforge.net/gazebo/xmlschema/#model"
 	xmlns:sensor="http://playerstage.sourceforge.net/gazebo/xmlschema/#sensor"
 	xmlns:body="http://playerstage.sourceforge.net/gazebo/xmlschema/#body"
-	xmlns:geom="http://playerstage.sourceforge.net/gazebo/xmlschema/#geom"
-	xmlns:joint="http://playerstage.sourceforge.net/gazebo/xmlschema/#joint"
+    xmlns:geom="http://playerstage.sourceforge.net/gazebo/xmlschema/#geom"
+    xmlns:joint="http://playerstage.sourceforge.net/gazebo/xmlschema/#joint"
 	xmlns:controller="http://playerstage.sourceforge.net/gazebo/xmlschema/#controller"
 	xmlns:interface="http://playerstage.sourceforge.net/gazebo/xmlschema/#interface"
 	xmlns:rendering="http://playerstage.sourceforge.net/gazebo/xmlschema/#rendering"
-	xmlns:renderable="http://playerstage.sourceforge.net/gazebo/xmlschema/#renderable"
-	xmlns:physics="http://playerstage.sourceforge.net/gazebo/xmlschema/#physics"
+    xmlns:renderable="http://playerstage.sourceforge.net/gazebo/xmlschema/#renderable"
+    xmlns:physics="http://playerstage.sourceforge.net/gazebo/xmlschema/#physics"
 	xmlns:xacro="http://ros.org/wiki/xacro">
 <xacro:include filename="$(find kinova_description)/urdf/kinova_inertial.xacro" />
@@ -31,5 +31,5 @@
                 <geometry>
                     <mesh
-                        filename="package://kinova_description/meshes/${ring_mesh}.STL"/>
+                        filename="package://kinova_description/meshes/${ring_mesh}.dae"/>
                 </geometry>
              </visual>
@@ -67,16 +67,5 @@
   </xacro:macro>
     <xacro:macro name="kinova_virtual_link" params="link_name">
-        <link name="${link_name}">
-            <!--visual>
-                <geometry>
-                    <box size = "0.01 0.01 0.01"/>
-                </geometry>
-            </visual>
-            <collision>
-                <geometry>
-                    <box size = "0.01 0.01 0.01"/>
-                </geometry>
-            </collision-->
-        </link>
+        <link name="${link_name}"/>
     </xacro:macro>
     <xacro:macro name="kinova_virtual_joint" params="joint_name type parent child joint_axis_xyz joint_origin_xyz joint_origin_rpy joint_lower_limit joint_upper_limit">

File: kinova-ros/kinova_description/urdf/m1n4s200_standalone.xacro (robot description, xacro)
@@ -3,38 +3,17 @@
 <robot xmlns:xi="http://www.w3.org/2001/XInclude"
 	xmlns:gazebo="http://playerstage.sourceforge.net/gazebo/xmlschema/#gz"
-	xmlns:model="http://playerstage.sourceforge.net/gazebo/xmlschema/#model"
+    xmlns:model="http://playerstage.sourceforge.net/gazebo/xmlschema/#model"
 	xmlns:sensor="http://playerstage.sourceforge.net/gazebo/xmlschema/#sensor"
 	xmlns:body="http://playerstage.sourceforge.net/gazebo/xmlschema/#body"
-	xmlns:geom="http://playerstage.sourceforge.net/gazebo/xmlschema/#geom"
-	xmlns:joint="http://playerstage.sourceforge.net/gazebo/xmlschema/#joint"
+    xmlns:geom="http://playerstage.sourceforge.net/gazebo/xmlschema/#geom"
+    xmlns:joint="http://playerstage.sourceforge.net/gazebo/xmlschema/#joint"
 	xmlns:controller="http://playerstage.sourceforge.net/gazebo/xmlschema/#controller"
 	xmlns:interface="http://playerstage.sourceforge.net/gazebo/xmlschema/#interface"
 	xmlns:rendering="http://playerstage.sourceforge.net/gazebo/xmlschema/#rendering"
-	xmlns:renderable="http://playerstage.sourceforge.net/gazebo/xmlschema/#renderable"
-	xmlns:physics="http://playerstage.sourceforge.net/gazebo/xmlschema/#physics"
+    xmlns:renderable="http://playerstage.sourceforge.net/gazebo/xmlschema/#renderable"
+    xmlns:physics="http://playerstage.sourceforge.net/gazebo/xmlschema/#physics"
 	xmlns:xacro="http://ros.org/wiki/xacro" name="m1n4s200">
   <xacro:include filename="$(find kinova_description)/urdf/m1n4s200.xacro"/>
-  <link name="root">
-    <visual>
-      <origin xyz="0 0 0" rpy="0 0 0" />
-      <geometry>
-        <box size = "0.01 0.01 0.01"/>
-      </geometry>
-    <!--<material name="Black" /> -->
-    </visual>
-    <collision>
-      <origin xyz="0 0 0" rpy="0 0 0" />
-      <geometry>
-        <box size = "0.01 0.01 0.01"/>
-      </geometry>
-    </collision>
-  </link>
-  <!-- for gazebo -->
-  <link name="world"/>
-  <joint name="connect_root_and_world" type="fixed">
-    <child link="root" />
-    <parent link="world" />
-    <origin xyz="0 0 0" rpy="0 0 0" />
-  </joint>
+  <link name="root"/>
   <xacro:property name="robot_root" value="root" />
   <xacro:m1n4s200  base_parent="${robot_root}"/>

File: kinova-ros/kinova_description/urdf/m1n6s200_standalone.xacro (robot description, xacro)
@@ -3,38 +3,17 @@
 <robot xmlns:xi="http://www.w3.org/2001/XInclude"
 	xmlns:gazebo="http://playerstage.sourceforge.net/gazebo/xmlschema/#gz"
-	xmlns:model="http://playerstage.sourceforge.net/gazebo/xmlschema/#model"
+    xmlns:model="http://playerstage.sourceforge.net/gazebo/xmlschema/#model"
 	xmlns:sensor="http://playerstage.sourceforge.net/gazebo/xmlschema/#sensor"
 	xmlns:body="http://playerstage.sourceforge.net/gazebo/xmlschema/#body"
-	xmlns:geom="http://playerstage.sourceforge.net/gazebo/xmlschema/#geom"
-	xmlns:joint="http://playerstage.sourceforge.net/gazebo/xmlschema/#joint"
+    xmlns:geom="http://playerstage.sourceforge.net/gazebo/xmlschema/#geom"
+    xmlns:joint="http://playerstage.sourceforge.net/gazebo/xmlschema/#joint"
 	xmlns:controller="http://playerstage.sourceforge.net/gazebo/xmlschema/#controller"
 	xmlns:interface="http://playerstage.sourceforge.net/gazebo/xmlschema/#interface"
 	xmlns:rendering="http://playerstage.sourceforge.net/gazebo/xmlschema/#rendering"
-	xmlns:renderable="http://playerstage.sourceforge.net/gazebo/xmlschema/#renderable"
-	xmlns:physics="http://playerstage.sourceforge.net/gazebo/xmlschema/#physics"
+    xmlns:renderable="http://playerstage.sourceforge.net/gazebo/xmlschema/#renderable"
+    xmlns:physics="http://playerstage.sourceforge.net/gazebo/xmlschema/#physics"
 	xmlns:xacro="http://ros.org/wiki/xacro" name="m1n6s200">
   <xacro:include filename="$(find kinova_description)/urdf/m1n6s200.xacro"/>
-  <link name="root">
-    <visual>
-      <origin xyz="0 0 0" rpy="0 0 0" />
-      <geometry>
-        <box size = "0.01 0.01 0.01"/>
-      </geometry>
-    <!--<material name="Black" /> -->
-    </visual>
-    <collision>
-      <origin xyz="0 0 0" rpy="0 0 0" />
-      <geometry>
-        <box size = "0.01 0.01 0.01"/>
-      </geometry>
-    </collision>
-  </link>
-  <!-- for gazebo -->
-  <link name="world"/>
-  <joint name="connect_root_and_world" type="fixed">
-    <child link="root" />
-    <parent link="world" />
-    <origin xyz="0 0 0" rpy="0 0 0" />
-  </joint>
+  <link name="root"/>
   <xacro:property name="robot_root" value="root" />
   <xacro:m1n6s200  base_parent="${robot_root}"/>
