Commit message: we can use moveit to control oarbot in gazebo

File: oarbot-ros/oarbot_description/robot/oarbot-old.urdf.xacro (robot description, xacro)
@@ -1,30 +1,1970 @@
-<?xml version="1.0"?>
-<robot name="summit_xl" xmlns:xacro="http://www.ros.org/wiki/xacro">
-	<!-- Import summit XL wheels -->
-	<xacro:include filename="$(find oarbot_description)/urdf/wheels/omni_wheel.urdf.xacro" />
-	<xacro:include filename="$(find oarbot_description)/urdf/base/oarbot_base.urdf.xacro" />
-	<xacro:include filename="$(find kinova_description)/urdf/j2n6s300.xacro" />
-	<!-- Wheel parameters -->
-	<xacro:property name="wheel_offset_x" value="0.2225" />    <!-- x,y,z in translation from base_link to the center of the wheel -->
-	<xacro:property name="wheel_offset_y" value="0.2045" />
-	<xacro:property name="wheel_offset_z" value="0.0" />
-	<xacro:macro name="robot">
-		<xacro:summit_base/>
-		<xacro:omni_wheel prefix="summit_front_right" parent="summit_base_link" reflect="false">
-			<origin xyz="${wheel_offset_x} -${wheel_offset_y} ${wheel_offset_z}" rpy="0 0 0"/>
-		</xacro:omni_wheel>
-		<xacro:omni_wheel prefix="summit_front_left" parent="summit_base_link" reflect="true">
-			<origin xyz="${wheel_offset_x} ${wheel_offset_y} ${wheel_offset_z}" rpy="0 0 0"/>
-		</xacro:omni_wheel>
-		<xacro:omni_wheel prefix="summit_back_left" parent="summit_base_link" reflect="true">
-			<origin xyz="-${wheel_offset_x} ${wheel_offset_y} ${wheel_offset_z}" rpy="0 0 0"/>
-		</xacro:omni_wheel>
-		<xacro:omni_wheel prefix="summit_back_right" parent="summit_base_link" reflect="false">
-			<origin xyz="-${wheel_offset_x} -${wheel_offset_y} ${wheel_offset_z}" rpy="0 0 0"/>
-		</xacro:omni_wheel>
-		<xacro:j2n6s300 prefix="j2n6s300" base_parent="support">
-		</xacro:j2n6s300>
-		<xacro:omni_steering />
-   </xacro:macro>
-   <xacro:robot/>
+<?xml version="1.0" ?>
+<!-- =================================================================================== -->
+<!-- |    This document was autogenerated by xacro from /home/ruijie/kinova_ws/src/oarbot-ros/oarbot_description/robot/oarbot.urdf.xacro | -->
+<!-- |    EDITING THIS FILE BY HAND IS NOT RECOMMENDED                                 | -->
+<!-- =================================================================================== -->
+<robot name="summit_xl" xmlns:body="http://playerstage.sourceforge.net/gazebo/xmlschema/#body" xmlns:controller="http://playerstage.sourceforge.net/gazebo/xmlschema/#controller" xmlns:gazebo="http://playerstage.sourceforge.net/gazebo/xmlschema/#gz" xmlns:geom="http://playerstage.sourceforge.net/gazebo/xmlschema/#geom" xmlns:interface="http://playerstage.sourceforge.net/gazebo/xmlschema/#interface" xmlns:joint="http://playerstage.sourceforge.net/gazebo/xmlschema/#joint" xmlns:model="http://playerstage.sourceforge.net/gazebo/xmlschema/#model" xmlns:physics="http://playerstage.sourceforge.net/gazebo/xmlschema/#physics" xmlns:renderable="http://playerstage.sourceforge.net/gazebo/xmlschema/#renderable" xmlns:rendering="http://playerstage.sourceforge.net/gazebo/xmlschema/#rendering" xmlns:sensor="http://playerstage.sourceforge.net/gazebo/xmlschema/#sensor" xmlns:xacro="http://www.ros.org/wiki/xacro" xmlns:xi="http://www.w3.org/2001/XInclude">
+    <!-- in kg-->
+    <!-- links      		mesh_no
+   base           		0
+   shoulder       		1
+   arm            		2
+   forearm        		3
+   wrist          		4
+   arm_mico       		5
+   arm_half1 (7dof)		6
+   arm_half2 (7dof)		7
+   wrist_spherical_1  8
+   wrist_spherical_2  9
+   hand 3 finger  		55
+   hand_2finger   		56
+   finger_proximal		57
+   finger_distal      58
+-->
+    <!-- links      		mesh_no
+   base           		0
+   shoulder       		1
+   arm            		2
+   forearm        		3
+   wrist          		4
+   arm_mico       		5
+   arm_half1 (7dof)		6
+   arm_half2 (7dof)		7
+   wrist_spherical_1  8
+   wrist_spherical_2  9
+   hand 3 finger  		55
+   hand_2finger   		56
+   finger_proximal		57
+   finger_distal      58
+-->
+    <!-- BASE FOOTPRINT -->
+    <link name="summit_base_footprint">
+        <visual>
+            <origin rpy="0 0 0" xyz="0 0 0" />
+            <geometry>
+                <box size="0.001 0.001 0.001" />
+            </geometry>
+        </visual>
+    </link>
+    <joint name="summit_base_footprint_joint" type="fixed">
+        <origin rpy="0 0 0" xyz="0 0 0.127" />
+        <!-- ${wheel_radius} property must be defined inside wheel description -->
+        <parent link="summit_base_footprint" />
+        <child link="summit_base_link" />
+    </joint>
+    <!-- BASE_LINK -->
+    <link name="summit_base_link">
+<inertial>
+            <mass value="125.0" />
+            <origin xyz="0 0 0" />
+            <inertia ixx="1.391" ixy="0.004" ixz="0.0" iyy="6.853" iyz="0.0" izz="6.125" />
+        </inertial>
+        <visual>
+            <origin rpy="0 0 0" xyz="0 0 0" />
+            <geometry>
+                <mesh filename="package://oarbot_description/meshes/base/summit_base.dae" />
+            </geometry>
+            <material name="darkgrey">
+                <color rgba="0.1 0.1 0.1 1" />
+            </material>
+        </visual>
+        <collision>
+            <origin rpy="0 0 0 " xyz="0 0 0" />
+            <geometry>
+                <mesh filename="package://oarbot_description/meshes/base/summit_base.dae" />
+            </geometry>
+        </collision>
+    </link>
+    <!-- for kinova arm support part -->
+    <material name="white">
+        <color rgba="1 1 1 1" />
+    </material>
+    <link name="support">
+        <visual>
+            <geometry>
+                <box size="0.15 0.15 0.3" />
+            </geometry>
+            <origin rpy="0 0 0" xyz="0 0 0" />
+            <material name="white" />
+        </visual>
+        <collision>
+            <geometry>
+                <box size="0.15 0.15 0.3" />
+            </geometry>
+        </collision>
+<inertial>
+            <mass value="0.1" />
+            <inertia ixx="0.03" iyy="0.03" izz="0.03" ixy="0.0" ixz="0.0" iyz="0.0" />
+        </inertial>
+    </link>
+    <joint name="base_to_support" type="fixed">
+        <parent link="summit_base_link" />
+        <child link="support" />
+        <origin xyz="-0.22 0 0.3" />
+    </joint>
+    <joint name="summit_front_right_wheel_joint" type="continuous">
+        <parent link="summit_base_link" />
+        <child link="summit_front_right_wheel_link" />
+        <origin rpy="0 0 0" xyz="0.2225 -0.2045 0.0" />
+        <axis rpy="0 0 0" xyz="0 1 0" />
+        <limit effort="100" velocity="100" />
+        <joint_properties damping="0.0" friction="0.0" />
+    </joint>
+    <link name="summit_front_right_wheel_link">
+        <visual>
+            <origin rpy="0 0 0" xyz="0 0 0" />
+            <geometry>
+                <mesh filename="package://oarbot_description/meshes/wheels/omni_wheel_2.dae" />
+            </geometry>
+        </visual>
+        <collision>
+            <origin rpy="1.57079632679 0 0" xyz="0 0 0" />
+            <geometry>
+                <cylinder length="0.087" radius="0.127" />
+            </geometry>
+        </collision>
+<inertial>
+            <mass value="6.5" />
+            <origin xyz="0 0 0" />
+            <inertia ixx="0.0303095" ixy="0" ixz="0" iyy="0.05241925" iyz="0" izz="0.0303095" />
+        </inertial>
+    </link>
+    <!-- Transmission is important to link the joints and the controller (see summit_xl_control/config/summit_xl_control.yaml)-->
+    <transmission name="summit_front_right_wheel_joint_trans">
+        <type>transmission_interface/SimpleTransmission</type>
+        <joint name="summit_front_right_wheel_joint">
+            <hardwareInterface>hardware_interface/VelocityJointInterface</hardwareInterface>
+        </joint>
+        <actuator name="summit_front_right_wheel_joint_motor">
+            <mechanicalReduction>1</mechanicalReduction>
+        </actuator>
+    </transmission>
+    <gazebo reference="summit_front_right_wheel_link">
+        <mu1 value="1.0" />
+        <mu2 value="1.0" />
+        <kp value="10000000.0" />
+        <kd value="1.0" />
+        <fdir1 value="1 0 0" />
+        <turnGravityOff>false</turnGravityOff>
+    </gazebo>
+    <joint name="summit_front_left_wheel_joint" type="continuous">
+        <parent link="summit_base_link" />
+        <child link="summit_front_left_wheel_link" />
+        <origin rpy="0 0 0" xyz="0.2225 0.2045 0.0" />
+        <axis rpy="0 0 0" xyz="0 1 0" />
+        <limit effort="100" velocity="100" />
+        <joint_properties damping="0.0" friction="0.0" />
+    </joint>
+    <link name="summit_front_left_wheel_link">
+        <visual>
+            <origin rpy="0 0 0" xyz="0 0 0" />
+            <geometry>
+                <mesh filename="package://oarbot_description/meshes/wheels/omni_wheel_1.dae" />
+            </geometry>
+        </visual>
+        <collision>
+            <origin rpy="1.57079632679 0 0" xyz="0 0 0" />
+            <geometry>
+                <cylinder length="0.087" radius="0.127" />
+            </geometry>
+        </collision>
+<inertial>
+            <mass value="6.5" />
+            <origin xyz="0 0 0" />
+            <inertia ixx="0.0303095" ixy="0" ixz="0" iyy="0.05241925" iyz="0" izz="0.0303095" />
+        </inertial>
+    </link>
+    <!-- Transmission is important to link the joints and the controller (see summit_xl_control/config/summit_xl_control.yaml)-->
+    <transmission name="summit_front_left_wheel_joint_trans">
+        <type>transmission_interface/SimpleTransmission</type>
+        <joint name="summit_front_left_wheel_joint">
+            <hardwareInterface>hardware_interface/VelocityJointInterface</hardwareInterface>
+        </joint>
+        <actuator name="summit_front_left_wheel_joint_motor">
+            <mechanicalReduction>1</mechanicalReduction>
+        </actuator>
+    </transmission>
+    <gazebo reference="summit_front_left_wheel_link">
+        <mu1 value="1.0" />
+        <mu2 value="1.0" />
+        <kp value="10000000.0" />
+        <kd value="1.0" />
+        <fdir1 value="1 0 0" />
+        <turnGravityOff>false</turnGravityOff>
+    </gazebo>
+    <joint name="summit_back_left_wheel_joint" type="continuous">
+        <parent link="summit_base_link" />
+        <child link="summit_back_left_wheel_link" />
+        <origin rpy="0 0 0" xyz="-0.2225 0.2045 0.0" />
+        <axis rpy="0 0 0" xyz="0 1 0" />
+        <limit effort="100" velocity="100" />
+        <joint_properties damping="0.0" friction="0.0" />
+    </joint>
+    <link name="summit_back_left_wheel_link">
+        <visual>
+            <origin rpy="0 0 0" xyz="0 0 0" />
+            <geometry>
+                <mesh filename="package://oarbot_description/meshes/wheels/omni_wheel_1.dae" />
+            </geometry>
+        </visual>
+        <collision>
+            <origin rpy="1.57079632679 0 0" xyz="0 0 0" />
+            <geometry>
+                <cylinder length="0.087" radius="0.127" />
+            </geometry>
+        </collision>
+<inertial>
+            <mass value="6.5" />
+            <origin xyz="0 0 0" />
+            <inertia ixx="0.0303095" ixy="0" ixz="0" iyy="0.05241925" iyz="0" izz="0.0303095" />
+        </inertial>
+    </link>
+    <!-- Transmission is important to link the joints and the controller (see summit_xl_control/config/summit_xl_control.yaml)-->
+    <transmission name="summit_back_left_wheel_joint_trans">
+        <type>transmission_interface/SimpleTransmission</type>
+        <joint name="summit_back_left_wheel_joint">
+            <hardwareInterface>hardware_interface/VelocityJointInterface</hardwareInterface>
+        </joint>
+        <actuator name="summit_back_left_wheel_joint_motor">
+            <mechanicalReduction>1</mechanicalReduction>
+        </actuator>
+    </transmission>
+    <gazebo reference="summit_back_left_wheel_link">
+        <mu1 value="1.0" />
+        <mu2 value="1.0" />
+        <kp value="10000000.0" />
+        <kd value="1.0" />
+        <fdir1 value="1 0 0" />
+        <turnGravityOff>false</turnGravityOff>
+    </gazebo>
+    <joint name="summit_back_right_wheel_joint" type="continuous">
+        <parent link="summit_base_link" />
+        <child link="summit_back_right_wheel_link" />
+        <origin rpy="0 0 0" xyz="-0.2225 -0.2045 0.0" />
+        <axis rpy="0 0 0" xyz="0 1 0" />
+        <limit effort="100" velocity="100" />
+        <joint_properties damping="0.0" friction="0.0" />
+    </joint>
+    <link name="summit_back_right_wheel_link">
+        <visual>
+            <origin rpy="0 0 0" xyz="0 0 0" />
+            <geometry>
+                <mesh filename="package://oarbot_description/meshes/wheels/omni_wheel_2.dae" />
+            </geometry>
+        </visual>
+        <collision>
+            <origin rpy="1.57079632679 0 0" xyz="0 0 0" />
+            <geometry>
+                <cylinder length="0.087" radius="0.127" />
+            </geometry>
+        </collision>
+<inertial>
+            <mass value="6.5" />
+            <origin xyz="0 0 0" />
+            <inertia ixx="0.0303095" ixy="0" ixz="0" iyy="0.05241925" iyz="0" izz="0.0303095" />
+        </inertial>
+    </link>
+    <!-- Transmission is important to link the joints and the controller (see summit_xl_control/config/summit_xl_control.yaml)-->
+    <transmission name="summit_back_right_wheel_joint_trans">
+        <type>transmission_interface/SimpleTransmission</type>
+        <joint name="summit_back_right_wheel_joint">
+            <hardwareInterface>hardware_interface/VelocityJointInterface</hardwareInterface>
+        </joint>
+        <actuator name="summit_back_right_wheel_joint_motor">
+            <mechanicalReduction>1</mechanicalReduction>
+        </actuator>
+    </transmission>
+    <gazebo reference="summit_back_right_wheel_link">
+        <mu1 value="1.0" />
+        <mu2 value="1.0" />
+        <kp value="10000000.0" />
+        <kd value="1.0" />
+        <fdir1 value="1 0 0" />
+        <turnGravityOff>false</turnGravityOff>
+    </gazebo>
+    <!-- ros_control plugin -->
+    <gazebo>
+        <plugin filename="libgazebo_ros_control.so" name="gazebo_ros_control">
+            <robotNamespace>j2n6s300</robotNamespace>
+            <robotSimType>gazebo_ros_control/DefaultRobotHWSim</robotSimType>
+            <legacyModeNS>true</legacyModeNS>
+        </plugin>
+    </gazebo>
+    <link name="j2n6s300_link_base">
+        <visual>
+            <geometry>
+                <mesh filename="package://kinova_description/meshes/base.dae" />
+            </geometry>
+            <material name="carbon_fiber">
+                <color rgba="0.792156862745098 0.819607843137255 0.933333333333333 1" />
+            </material>
+        </visual>
+        <collision>
+            <geometry>
+                <mesh filename="package://kinova_description/meshes/base.dae" />
+            </geometry>
+        </collision>
+<inertial>
+            <mass value="0.46784" />
+            <origin rpy="0 0 0" xyz="0 0 0.1255" />
+            <inertia ixx="0.000951270861568" ixy="0" ixz="0" iyy="0.000951270861568" iyz="0" izz="0.000374272" />
+        </inertial>
+    </link>
+    <joint name="j2n6s300_joint_base" type="fixed">
+        <parent link="support" />
+        <child link="j2n6s300_link_base" />
+        <axis xyz="0 0 0" />
+        <limit effort="0" lower="0" upper="0" velocity="0" />
+        <origin rpy="0 0 0" xyz="0 0 0" />
+        <dynamics damping="0.0" friction="0.0" />
+    </joint>
+    <link name="j2n6s300_link_1">
+        <visual>
+            <geometry>
+                <mesh filename="package://kinova_description/meshes/shoulder.dae" />
+            </geometry>
+            <material name="carbon_fiber">
+                <color rgba="0.792156862745098 0.819607843137255 0.933333333333333 1" />
+            </material>
+        </visual>
+        <visual>
+            <geometry>
+                <mesh filename="package://kinova_description/meshes/ring_big.dae" />
+            </geometry>
+        </visual>
+        <collision>
+            <geometry>
+                <mesh filename="package://kinova_description/meshes/shoulder.dae" />
+            </geometry>
+        </collision>
+<inertial>
+            <mass value="0.7477" />
+            <origin xyz="0 -0.002 -0.0605" />
+            <inertia ixx="0.00152031725204" ixy="0" ixz="0" iyy="0.00152031725204" iyz="0" izz="0.00059816" />
+        </inertial>
+    </link>
+    <joint name="j2n6s300_joint_1" type="continuous">
+        <parent link="j2n6s300_link_base" />
+        <child link="j2n6s300_link_1" />
+        <axis xyz="0 0 1" />
+        <limit effort="40" lower="-6.28318530718" upper="6.28318530718" velocity="0.628318530718" />
+        <origin rpy="0 3.14159265359 0" xyz="0 0 0.15675" />
+        <dynamics damping="0.0" friction="0.0" />
+    </joint>
+    <transmission name="j2n6s300_joint_1_trans">
+        <type>transmission_interface/SimpleTransmission</type>
+        <joint name="j2n6s300_joint_1">
+            <hardwareInterface>hardware_interface/EffortJointInterface</hardwareInterface>
+        </joint>
+        <actuator name="j2n6s300_joint_1_actuator">
+            <hardwareInterface>hardware_interface/EffortJointInterface</hardwareInterface>
+            <mechanicalReduction>160</mechanicalReduction>
+        </actuator>
+    </transmission>
+    <!--For torque sensing in simulation-->
+    <gazebo reference="j2n6s300_joint_1">
+        <provideFeedback>true</provideFeedback>
+    </gazebo>
+    <gazebo>
+        <plugin filename="libgazebo_ros_ft_sensor.so" name="ft_sensor">
+            <updateRate>30.0</updateRate>
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